Commit message: working_version

File: my_robot/urdf/my_robot.xacro (robot description, xacro)
@@ -11,5 +11,5 @@
       <pose>0 0 0.1 0 0 0</pose>
       <inertial>
-        <mass value="15.0"/>
+        <mass value="10.0"/>
         <origin xyz="0.0 0 0" rpy=" 0 0 0"/>
         <inertia
@@ -34,5 +34,10 @@
         </material>
       </visual>
-      <collision name='back_caster_collision'>
+  <link name='back_caster_collision'>
+    <inertial>
+       <mass value="100.0"/>
+       <inertia ixx="0.1" ixy="0" ixz="0" iyy="0.1" iyz="0" izz="0.1"/>
+    </inertial>
+      <collision>
         <origin xyz="-0.15 0 -0.05" rpy=" 0 0 0"/>
         <geometry>
@@ -40,5 +45,5 @@
         </geometry>
       </collision>
-      <visual name='back_caster_visual'>
+      <visual>
         <origin xyz="-0.15 0 -0.05" rpy=" 0 0 0"/>
         <geometry>
@@ -49,5 +54,11 @@
         </material>
       </visual>
-      <collision name='front_caster_collision'>
+    </link>
+ <link name='front_caster_collision'>
+    <inertial>
+       <mass value="100.0"/>
+       <inertia ixx="0.1" ixy="0" ixz="0" iyy="0.1" iyz="0" izz="0.1"/>
+    </inertial>
+      <collision>
         <origin xyz="0.15 0 -0.05" rpy=" 0 0 0"/>
         <geometry>
@@ -55,5 +66,5 @@
         </geometry>
       </collision>
-      <visual name='front_caster_visual'>
+      <visual>
         <origin xyz="0.15 0 -0.05" rpy=" 0 0 0"/>
         <geometry>
@@ -68,7 +79,8 @@
       <material>Gazebo/Blue</material>
   </gazebo>
+</link>
   <link name="left_wheel">
     <inertial>
-       <mass value="15.0"/>
+       <mass value="100.0"/>
        <origin xyz="0 0 0" rpy=" 0 1.5707 1.5707"/>
        <inertia ixx="0.1" ixy="0" ixz="0" iyy="0.1" iyz="0" izz="0.1"/>
@@ -103,5 +115,5 @@
   <link name="right_wheel">
     <inertial>
-       <mass value="15.0"/>
+       <mass value="100.0"/>
        <origin xyz="0 0 0" rpy=" 0 1.5707 1.5707"/>
        <inertia ixx="0.1" ixy="0" ixz="0" iyy="0.1" iyz="0" izz="0.1"/>
